File: biosemicard-exp.kicad_sch (KiCad schematic)
At the start: 10 parts, among them J1 Conn_01x12_Pin, J2 Conn_01x08_Pin, U2 74HC151D

Commit message: added simulation
Parts:
- removed C42: 100n, symbol Device:C
- removed C43: 2.2u, symbol Device:C
- removed FB10, FB9: FerriteBead, Inductor_SMD:L_0402_1005Metric, symbol Device:FerriteBead
- removed V3: 2.5, symbol Simulation_SPICE:VDC
Connections:
- net +2V5: now also J2.2 (Pin_2)
- net +2V93: now also J1.12 (Pin_12)
- net 0 renamed GNDD
- net GNDD: no longer J1.9 (Pin_9)
- net S0: no longer names the net of J2.5 (Pin_5), U2.11 (S0)
- net S1: no longer names the net of J2.6 (Pin_6), U2.10 (S1)
- net S2: no longer names the net of J2.7 (Pin_7), U2.9 (S2)
- new net GND: J1.9 (Pin_9)
Other:
- note added: "DATA"
- moved on the sheet: C3
