File: _autosave-biosemicard.kicad_pcb (KiCad board)
At the start: 4 copper layers, 67 x 38 mm, 144 parts, among them J1 Conn_01x26_Pin, U1 OPA2188AIDR, U10 OPA2188AIDR, U11 ADS1254E, U12 OPA2188AIDR, U13 ADS1254E, U14 OPA2188AIDR, U15 ADS1254E, U16 OPA2188AIDR, U17 ADS1254E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

Commit message: layout v2
Routing:
- added copper zone on F.Cu, net -2V048
- added copper zone on B.Cu, net GNDD
Changed lines of the file:
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@@
+		(net 2)
+		(net_name "-2V048")
+		(layer "F.Cu")
+		(hatch edge 0.5)
+		(priority 2)
+		(connect_pads yes
+			(clearance 0.5)
+		)
+		(min_thickness 0.25)
+		(filled_areas_thickness no)
+		(fill yes
+			(thermal_gap 0.5)
+			(thermal_bridge_width 0.5)
+		)
+		(polygon
+			(pts
+				(xy 28.5 56.15) (xy 28.4 93.9) (xy 95.15 93.95) (xy 95.1 56)
+			)
+		)
+	)
+	(zone
 		(net 2)
 		(net_name "-2V048")
@@
 			)
 		)
+	)
+	(zone
+		(net 6)
+		(net_name "GNDD")
+		(layer "B.Cu")
+		(hatch edge 0.5)
+		(priority 3)
+		(connect_pads yes
+			(clearance 0.5)
+		)
+		(min_thickness 0.25)
+		(filled_areas_thickness no)
+		(fill yes
+			(thermal_gap 0.5)
+			(thermal_bridge_width 0.5)
+		)
+		(polygon
+			(pts
+				(xy 28.35 56.25) (xy 28.35 93.95) (xy 94.9 93.85) (xy 94.95 56.25) (xy 28.3 56.05)
+			)
+		)
